File: UnicornBoard.kicad_pcb (KiCad board)
At the start: 2 copper layers, 33.8 x 39.7 mm, 37 parts, among them J2 USB_B_Micro, SW1 SW_Push, U1 ATSAMD21E18A-AU, U2 AP2112K-3.3

Commit message: Candy the Catacorn
Parts:
- removed J2: USB_B_Micro, Connector_USB:USB_Micro-B_GCT_USB3076-30-A
- added BT1: Battery, Connector_JST:JST_PH_S2B-PH-SM4-TB_1x02-1MP_P2.00mm_Horizontal, B.Cu at (228.6, 108.0)
- added D50: D_Schottky, Diode_SMD:D_SOD-123F, B.Cu at (235.6, 114.3)
- added H1: MountingHole, MountingHole:MountingHole_2.2mm_M2_ISO7380_Pad, F.Cu at (220.2, 135.5)
- added H2: MountingHole, MountingHole:MountingHole_2.2mm_M2_ISO7380_Pad, F.Cu at (237.0, 134.5)
- added USB: USB_B_Micro, Connector_USB:USB_Micro-B_GCT_USB3076-30-A, B.Cu at (229.1, 150.1)
- C1: renamed from C5; value C -> 1 uF C
- C2: renamed from C6; value C -> 10 uF C
- C3: renamed from C7; value C -> 10 uF C; moved to B.Cu
- C4: renamed from C8; value C -> 1 uF C
- D4: renamed from Tail0; footprint LED_SMD:LED_0402_1005Metric -> LED_SMD:LED_0805_2012Metric_Pad1.15x1.40mm_HandSolder
- D5: renamed from Tail2; footprint LED_SMD:LED_0402_1005Metric -> LED_SMD:LED_0805_2012Metric_Pad1.15x1.40mm_HandSolder
- D51: renamed from D7; footprint Diode_SMD:D_SOT-23_ANK -> Diode_SMD:D_SOD-123F
- D6: renamed from Tail1; footprint LED_SMD:LED_0402_1005Metric -> LED_SMD:LED_0805_2012Metric_Pad1.15x1.40mm_HandSolder
- D7: renamed from D6; footprint LED_SMD:LED_0402_1005Metric -> LED_SMD:LED_0805_2012Metric_Pad1.15x1.40mm_HandSolder
- D8: renamed from D1; footprint LED_SMD:LED_0402_1005Metric -> LED_SMD:LED_0805_2012Metric_Pad1.15x1.40mm_HandSolder
- D9: renamed from D2; footprint LED_SMD:LED_0402_1005Metric -> LED_SMD:LED_0805_2012Metric_Pad1.15x1.40mm_HandSolder
- R0: renamed from R1; value R -> 180R
- R1: renamed from R3; value R -> 180R
- R2: renamed from R4; value R -> 30R; footprint Resistor_SMD:R_0805_2012Metric_Pad1.15x1.40mm_HandSolder -> Resistor_SMD:R_1206_3216Metric_Pad1.42x1.75mm_HandSolder
- R3: renamed from R5; value R -> 30R; footprint Resistor_SMD:R_0805_2012Metric_Pad1.15x1.40mm_HandSolder -> Resistor_SMD:R_1206_3216Metric_Pad1.42x1.75mm_HandSolder
- R4: renamed from R6; value R -> 100R; footprint Resistor_SMD:R_0402_1005Metric -> Resistor_SMD:R_0603_1608Metric_Pad1.05x0.95mm_HandSolder
- R5: renamed from R7; value R -> 100R; footprint Resistor_SMD:R_0402_1005Metric -> Resistor_SMD:R_0603_1608Metric_Pad1.05x0.95mm_HandSolder
- R6: renamed from R8; value R -> 100R; footprint Resistor_SMD:R_0402_1005Metric -> Resistor_SMD:R_0603_1608Metric_Pad1.05x0.95mm_HandSolder
- R7: renamed from R2; value R -> 330R; footprint Resistor_SMD:R_0402_1005Metric -> Resistor_SMD:R_0805_2012Metric_Pad1.15x1.40mm_HandSolder
- R8: renamed from R9; value R -> 330R; footprint Resistor_SMD:R_0402_1005Metric -> Resistor_SMD:R_0805_2012Metric_Pad1.15x1.40mm_HandSolder
- R9: renamed from R10; value R -> 330R; footprint Resistor_SMD:R_0402_1005Metric -> Resistor_SMD:R_0805_2012Metric_Pad1.15x1.40mm_HandSolder
- moved Touch1 85.4 mm to (243.3, 103.3)
- moved GND 69.6 mm to (237.5, 117.6)
- moved 3V3 68.6 mm to (234.4, 117.6)
- moved C4 66.2 mm to (237.2, 120.9), turned to 90 degrees
- moved D5 63.2 mm to (250.1, 127.8), turned to 46 degrees
- moved D6 63.0 mm to (246.6, 134.5), turned to 80 degrees
- moved R5 62.8 mm to (249.6, 128.3), turned to 45 degrees
- moved R6 62.7 mm to (246.4, 134.6), turned to 81 degrees
- moved D4 62.6 mm to (244.1, 143.4), turned to 40 degrees
- moved R0 62.2 mm to (240.5, 115.6)
- moved R4 61.8 mm to (243.2, 144.1)
- moved D9 61.6 mm to (240.4, 149.9)
- moved R3 61.5 mm to (232.4, 144.8)
- moved R9 60.0 mm to (238.5, 147.1)
- moved D0 59.7 mm to (241.3, 112.8), turned to 278 degrees
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- renumbered D5 to D0, D3 to D1, Paw0 to D2, Paw1 to D3, Dot0 to Dot2, SW1 to Reset, Touch2 to Touch1, Touch1 to Touch2
Connections:
- C2 pad 1: +3V3 -> GND
- C2 pad 2: GND -> +3V3
- D1 pad 2: Net-(D3-Pad2) (its old number) -> Net-(D1-Pad2)
- D7 pad 2: Net-(D6-Pad2) (its old number) -> Net-(D7-Pad2)
- R0 pad 1: Net-(R1-Pad1) -> Net-(R0-Pad1)
- R1 pad 1: Net-(D3-Pad2) (its old number) -> Net-(R0-Pad1)
- R1 pad 2: Net-(R1-Pad1) -> Net-(D1-Pad2)
- R7 pad 2: Net-(D6-Pad2) (its old number) -> Net-(D7-Pad2)
- R8 pad 1: Net-(D6-Pad2) (its old number) -> +3V3
- R9 pad 1: Net-(D6-Pad2) (its old number) -> +3V3
- U1 pad 13: Net-(R1-Pad1) -> Net-(R0-Pad1)
Routing:
- net Net-(D6-Pad2) (its old number): track 57.7 -> 0.00 mm, vias 1 -> 0
- net +3V3: track 73.8 -> 125.3 mm, vias 2 -> 7
- net Net-(R0-Pad1): track 0.00 -> 35.0 mm, vias 0 -> 4
- net Net-(C3-Pad1): track 13.1 -> 40.8 mm, vias 1 -> 0
- net Net-(R2-Pad2): track 35.4 -> 60.8 mm, vias 4 -> 6
- net Net-(R1-Pad1): track 23.0 -> 0.00 mm
- net Net-(J2-Pad6): track 21.7 -> 0.00 mm
- net GND: track 155.5 -> 137.9 mm, vias 9 -> 24
- net Net-(J5-Pad6): track 0.00 -> 13.5 mm
- net Net-(Dot2-Pad2): track 6.64 -> 19.9 mm
- net Net-(Touch1-Pad1): track 9.34 -> 21.3 mm
- net Net-(R4-Pad1): track 64.9 -> 76.6 mm
- net Net-(Dot1-Pad1): track 6.71 -> 15.6 mm
- net Net-(Dot1-Pad2): track 6.71 -> 14.4 mm
- net +BATT: track 0.00 -> 5.77 mm
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Other:
- board size 33.8 x 39.7 mm -> 48.1 x 58.1 mm
- board text added: "Candy the Catacorn by @GalaxyAllieCat #BadgeLife 2020"
- board text removed: "@GalaxyAllieCat"

Commit message: Added inspirational quote to back silkscreen
Other:
- board text added: ""If you believe it, you achieve it!""
Changed lines of the file:
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@@
   (general
     (thickness 1.6)
-    (drawings 1057)
+    (drawings 1058)
     (tracks 425)
     (zones 0)
@@
   )
   (setup
-    (last_trace_width 0.3)
+    (last_trace_width 0.25)
     (user_trace_width 0.2)
     (user_trace_width 0.22)
@@
       (plotinvisibletext false)
       (padsonsilk false)
-      (subtractmaskfromsilk false)
+      (subtractmaskfromsilk true)
       (outputformat 1)
       (mirror false)
-      (drillshape 1)
+      (drillshape 0)
       (scaleselection 1)
-      (outputdirectory ""))
+      (outputdirectory "/home/allie/Documents/UnicornGerbers/"))
   )
   (net 0 "")
@@
       (net 31 "Net-(Touch2-Pad1)"))
   )
+  (gr_text "\"If you believe it,\nyou achieve it!\"" (at 239.014 125.857) (layer B.SilkS)
+    (effects (font (size 0.8 0.8) (thickness 0.15) italic) (justify mirror))
+  )
   (gr_line (start 223.015301 102.330012) (end 223.015301 102.330012) (layer Edge.Cuts) (width 0.36023))
   (gr_line (start 223.015301 102.330012) (end 223.015301 102.330012) (layer Edge.Cuts) (width 0.36023))
@@
   (segment (start 216.61444 113.58556) (end 216.916 113.284) (width 0.25) (layer F.Cu) (net 43))
   (segment (start 215.445762 113.58556) (end 216.61444 113.58556) (width 0.25) (layer F.Cu) (net 43))
-  (segment (start 223.683 118.745) (end 223.842 118.904) (width 0.22) (layer B.Cu) (net 49))
-  (segment (start 220.98 118.745) (end 223.683 118.745) (width 0.22) (layer B.Cu) (net 49))
-  (segment (start 220.98 116.205) (end 220.98 117.094) (width 0.22) (layer B.Cu) (net 50))
-  (segment (start 221.99 118.104) (end 223.842 118.104) (width 0.22) (layer B.Cu) (net 50))
-  (segment (start 220.98 117.094) (end 221.99 118.104) (width 0.22) (layer B.Cu) (net 50))
   (segment (start 233.934 121.876) (end 233.934 122.936) (width 0.22) (layer B.Cu) (net 44))
   (segment (start 232.342 121.304) (end 233.362 121.304) (width 0.22) (layer B.Cu) (net 44))
@@
   (segment (start 225.533 151.314) (end 226.258 151.314) (width 0.2) (layer B.Cu) (net 47))
   (segment (start 226.258 151.314) (end 226.788 150.784) (width 0.2) (layer B.Cu) (net 47))
+  (segment (start 223.683 118.745) (end 223.842 118.904) (width 0.22) (layer B.Cu) (net 49))
+  (segment (start 220.98 118.745) (end 223.683 118.745) (width 0.22) (layer B.Cu) (net 49))
+  (segment (start 220.98 116.205) (end 220.98 117.094) (width 0.22) (layer B.Cu) (net 50))
+  (segment (start 221.99 118.104) (end 223.842 118.104) (width 0.22) (layer B.Cu) (net 50))
+  (segment (start 220.98 117.094) (end 221.99 118.104) (width 0.22) (layer B.Cu) (net 50))
   (zone (net 30) (net_name "Net-(Touch1-Pad1)") (layer F.Cu) (hatch edge 0.508)
     (connect_pads yes (clearance 0.381))
