File: KiCad Project - Rev2 (RP2040 Base)/Candy-rev2/Candy-rev2.kicad_sch (KiCad schematic)
At the start: 2 parts

Commit message: thurs evening
Parts:
- added D? (x7): LED, symbol Device:LED
- added R? (x5): 1M, symbol Device:R
- added TP?: Nose, symbol Connector:TestPoint
- added TP? (x2): Right Ear, symbol Connector:TestPoint
- added TP?: Left Cheek, symbol Connector:TestPoint
- added TP?: Left Ear, symbol Connector:TestPoint
Connections:
- net VCC: now reaches D?.1 (VDD)
- net VCC: now also D?.1 (VDD)
- net EyeOut: now reaches D?.2 (DOUT)
- net GND: now reaches D?.3 (VSS)
- net GND: now also D?.3 (VSS), D?.1 (K), D?.1 (K), D?.1 (K), D?.1 (K), D?.1 (K), D?.1 (K), D?.1 (K), R?.2, R?.2, R?.2, R?.2, R?.2
- net at D?.4 (DIN): now also D?.2 (DOUT)
- net EyeIn: now reaches D?.4 (DIN)
- new net CheekL: R?.1, TP?.1
- new net CheekR: R?.1, TP?.1
- new net EarL: R?.1, TP?.1
- new net EarR: R?.1, TP?.1
- new net Front_LPaw: D?.2 (A)
- new net Front_RPaw: D?.2 (A)
- new net Nose: R?.1, TP?.1
- new net Rear_Paws: D?.2 (A), D?.2 (A)
- new net Tail_1: D?.2 (A)
- new net Tail_2: D?.2 (A)
- new net Tail_3: D?.2 (A)
Other:
- note added: "Eyes (WS2812)"
- note added: "Single-color LEDs"
- note added: "Touch Points"
- moved on the sheet: D?
